File: FeederShieldMega.brd (EAGLE design)
At the start: 86.4 x 53.3 mm, 44 parts, among them J1 Digital_0_7, J10 Power, J2 Analog, J3 Digital_8_13, J4 Analog, J5 Digital_0_7, J6 Digital_22_36, J7 Digital_23_37, J8 Digital_38_52, J9 Digital_39_53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

Commit message: Tweaks for v1.0 release
Parts:
- JP23: value N20 -> (none)
- JP24: value N21 -> (none)
- JP25: value N22 -> (none)
- JP26: value N23 -> (none)
Changed lines of the file:
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@@
 <element name="JP21" library="freetronics-jon" package="1X04" value="N18" x="53.34" y="15.24" rot="R90"/>
 <element name="JP22" library="freetronics-jon" package="1X04" value="N19" x="55.88" y="15.24" rot="R90"/>
-<element name="JP23" library="freetronics-jon" package="1X04" value="N20" x="63.5" y="15.24" rot="R90"/>
-<element name="JP24" library="freetronics-jon" package="1X04" value="N21" x="66.04" y="15.24" rot="R90"/>
-<element name="JP25" library="freetronics-jon" package="1X04" value="N22" x="68.58" y="15.24" rot="R90"/>
-<element name="JP26" library="freetronics-jon" package="1X04" value="N23" x="71.12" y="15.24" rot="R90"/>
+<element name="JP23" library="freetronics-jon" package="1X04" value="" x="63.5" y="15.24" rot="R90"/>
+<element name="JP24" library="freetronics-jon" package="1X04" value="" x="66.04" y="15.24" rot="R90"/>
+<element name="JP25" library="freetronics-jon" package="1X04" value="" x="68.58" y="15.24" rot="R90"/>
+<element name="JP26" library="freetronics-jon" package="1X04" value="" x="71.12" y="15.24" rot="R90"/>
 <element name="Q2" library="freetronics-master-v1.1" package="DPACK" value="NTD5867NLT4G" x="66.04" y="10.16" rot="R90"/>
 <element name="R1" library="freetronics-jon" package="0603" value="1K" x="73.66" y="7.62" rot="R90"/>
