File: FeederShieldMega.brd (EAGLE design)
At the start: 86.4 x 53.3 mm, 29 parts, among them J1 Digital_0_7, J10 Power, J11 M02X5-SHROUDED, J12 M02X5-SHROUDED, J13 M02X5-SHROUDED, J14 M02X5-SHROUDED, J15 M02X5-SHROUDED, J16 M02X5-SHROUDED, J2 Analog, J3 Digital_8_13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

Commit message: Added 5V 3A voltage regulator and removed 2 bulk decoupling caps for v3.0 release
Parts:
- removed C2, C3: 1000uF 25V, SuperHouse-DiscreteSemi:CPOL-RADIAL-5.08-10X18-FLAT
- removed JP27: (no value), SuperHouse-Connectors:1X02-P
- added MOD2: DC5V3A-SMT, SuperHouse-Regulators:DC5V3A-SMT
- C1: value 1000uF 25V -> 1000uF 16V
- moved LED1 12.7 mm to (24.1, 8.89), turned to 0 degrees
- moved R3 7.96 mm to (25.4, 28.7)
Connections:
- new net 5V_2: JP2.1, JP2.2
- net 5V: no longer C1.1, C2.1, C3.1, JP2.1, JP2.2, JP27.1
- net F_5V: now also C1.1, MOD2.3A, MOD2.3B; no longer JP27.2
- net GND: now also MOD2.1A, MOD2.1B, MOD2.4A, MOD2.4B; no longer C2.2, C3.2
- net VIN: now also MOD2.2A, MOD2.2B
Routing:
- net 5V: track 127.4 -> 13.9 mm
- net F_5V: track 107.1 -> 164.3 mm
- net VIN: track 0.00 -> 29.7 mm
- net N$5: track 3.12 -> 19.3 mm
- net F_GND: track 125.5 -> 121.0 mm
- net 5V_2: track 0.00 -> 2.54 mm
Other:
- board text added: "Copyright 2018-2020 SuperHouse Automation Released under the TAPR Open Hardware License: www.tapr.org/OHL"
- board text added: "MGRL0816 Feeder Shield"
- board text added: "Super House"
- board text added: "v3.0"
- board text added: "www.superhouse.tv/fsm"
- board text removed: "Copyright 2018-2020 Freetronics Pty Ltd Released under the TAPR Open Hardware License: www.tapr.org/OHL"
- board text removed: "PnP Feeder Shield"
- board text removed: "freetronics"
- board text removed: "v2.0"
- board text removed: "www.freetronics.com.au/fsm"
